File: WEMOS VER/wemos/wemos.kicad_pcb (KiCad board)
At the start: 2 copper layers, 50 x 60 mm, 27 parts, among them J1 9V BATT, J2 MOTOR 1, J3 MOTOR 2, SW1 RESET, SW2 ON/OFF, U1 WeMos D1 Mini, U2 L7805, U3 L293D

Commit message: work
pcb pdf revision
Parts:
- moved ? 0.40 mm to (74.0, 76.5)
Routing:
- net +9V: track 82.5 -> 83.6 mm
- net Net-(U1-D4): track 29.0 -> 29.8 mm
Other:
- board text added: "Bawah"
Changed lines of the file:
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@@
 	(footprint ""
 		(layer "F.Cu")
-		(at 73.66 76.708)
+		(at 74 76.5)
 		(property "Reference" ""
 			(at 0 0 0)
@@
 		(tags "TO-220-3 Vertical RM 2.54mm")
 		(property "Reference" "U2"
-			(at 2.54 -4.27 -90)
+			(at -3.88 -2.565 -90)
 			(layer "F.SilkS")
 			(effects
@@
 		)
 		(fp_text user "${REFERENCE}"
-			(at 2.54 -4.27 -90)
+			(at -3.88 -2.565 -90)
 			(layer "F.Fab")
 			(effects
@@
 		(layer "Edge.Cuts")
 	)
+	(gr_text "Bawah"
+		(at 76 35.5 0)
+		(layer "B.Cu")
+		(effects
+			(font
+				(size 1.5 1.5)
+				(thickness 0.3)
+				(bold yes)
+			)
+			(justify left bottom)
+		)
+	)
 	(gr_text "+"
 		(at 102.62 52.12 -90)
@@
 	(dimension
 		(type aligned)
-		(layer "User.1")
+		(layer "B.Cu")
 		(pts
 			(xy 105.62 98.62) (xy 105.62 38.62)
@@
 		(gr_text "60,0000 mm"
 			(at 117.97 68.62 90)
-			(layer "User.1")
+			(layer "B.Cu")
 			(effects
 				(font
@@
 	(dimension
 		(type aligned)
-		(layer "User.1")
+		(layer "B.Cu")
 		(pts
 			(xy 105.62 38.62) (xy 55.62 38.62)
@@
 		(gr_text "50,0000 mm"
 			(at 80.62 28.32 0)
-			(layer "User.1")
+			(layer "B.Cu")
 			(effects
 				(font
@@
 	)
 	(segment
+		(start 92.62 86.794886)
+		(end 94.5 84.914886)
+		(width 1)
+		(layer "B.Cu")
+		(net 3)
+	)
+	(segment
 		(start 60.62 87.62)
 		(end 62.62 89.62)
@@
 	)
 	(segment
-		(start 92.62 88.62)
-		(end 96.325114 84.914886)
-		(width 1)
-		(layer "B.Cu")
-		(net 3)
-	)
-	(segment
 		(start 96.62 78.12)
 		(end 96.62 84.914886)
@@
 	)
 	(segment
-		(start 96.325114 84.914886)
+		(start 94.5 84.914886)
 		(end 96.62 84.914886)
 		(width 1)
@@
 	)
 	(segment
+		(start 92.62 88.62)
+		(end 92.62 86.794886)
+		(width 1)
+		(layer "B.Cu")
+		(net 3)
+	)
+	(segment
 		(start 104.12 71.12)
 		(end 104.12 78.12)
@@
 	)
 	(segment
-		(start 84.804 73.12)
-		(end 78.74 67.056)
+		(start 86.868 73.406)
+		(end 85.09 73.406)
 		(width 0.5)
 		(layer "F.Cu")
@@
 	)
 	(segment
-		(start 85.62 73.12)
-		(end 84.804 73.12)
+		(start 85.09 73.406)
+		(end 78.74 67.056)
 		(width 0.5)
 		(layer "F.Cu")
@@
 	)
 	(segment
-		(start 89.12 83.62)
-		(end 75.62 83.62)
+		(start 86.868 73.406)
+		(end 88.392 73.406)
 		(width 0.5)
 		(layer "B.Cu")
@@
 	)
 	(segment
-		(start 78.18 59.93)
-		(end 69.205 59.93)
+		(start 91.62 81.12)
+		(end 89.12 83.62)
 		(width 0.5)
 		(layer "B.Cu")
@@
 	)
 	(segment
-		(start 75.62 83.62)
-		(end 74.46 84.78)
+		(start 78.18 59.93)
+		(end 69.205 59.93)
 		(width 0.5)
 		(layer "B.Cu")
@@
 	)
 	(segment
-		(start 91.62 81.12)
-		(end 89.12 83.62)
+		(start 91.62 76.634)
+		(end 91.62 81.12)
 		(width 0.5)
 		(layer "B.Cu")
@@
 	)
 	(segment
-		(start 88.106 73.12)
-		(end 91.62 76.634)
+		(start 89.12 83.62)
+		(end 75.62 83.62)
 		(width 0.5)
 		(layer "B.Cu")
@@
 	)
 	(segment
-		(start 78.74 60.49)
-		(end 78.18 59.93)
+		(start 88.392 73.406)
+		(end 91.62 76.634)
 		(width 0.5)
 		(layer "B.Cu")
@@
 	)
 	(segment
-		(start 85.62 73.12)
-		(end 88.106 73.12)
+		(start 78.74 60.49)
+		(end 78.18 59.93)
 		(width 0.5)
 		(layer "B.Cu")
@@
 	)
 	(segment
-		(start 91.62 76.634)
-		(end 91.62 81.12)
+		(start 75.62 83.62)
+		(end 74.46 84.78)
 		(width 0.5)
 		(layer "B.Cu")
@@
 	)
 	(segment
-		(start 73.12 76.62)
+		(start 74 54.5)
 		(end 73.12 53.62)
 		(width 0.5)
 		(layer "F.Cu")
+		(net 17)
+	)
+	(segment
+		(start 74 75.74)
+		(end 74 54.5)
+		(width 0.5)
+		(layer "F.Cu")
+		(net 17)
+	)
+	(segment
+		(start 73.12 76.62)
+		(end 74 75.74)
+		(width 0.5)
+		(layer "F.Cu")

Commit message: revisions
Parts:
- removed ? (x6): , 
- removed REF** (x6): SolderWire-0.5sqmm_1x01_D0.9mm_OD2.3mm, Connector_Wire:SolderWire-0.5sqmm_1x01_D0.9mm_OD2.3mm
- removed SW2: ON/OFF, Connector_PinSocket_2.54mm:PinSocket_1x03_P2.54mm_Vertical
Connections:
- J1 pad 1: Net-(J1-Pin_1) -> +9V
Routing:
- net GND: track 0.00 -> 31.8 mm, vias 0 -> 4
- net Net-(J1-Pin_1): track 31.1 -> 0.00 mm
- net +9V: track 83.6 -> 108.3 mm, vias 0 -> 2
- net Net-(J2-Pin_1): track 19.6 -> 22.0 mm
- net Net-(U1-D4): track 29.8 -> 31.4 mm, vias 0 -> 2
- net Net-(U1-SCL/D1): track 58.7 -> 57.8 mm, vias 0 -> 2
- net Net-(U1-SDA/D2): track 49.9 -> 49.1 mm, vias 0 -> 2
- net +5V: track 70.3 -> 70.5 mm, vias 0 -> 2
